File: KiCad/Guitar_Fx_Dev.kicad_pcb (KiCad board)
At the start: 2 copper layers, 95.6 x 99.4 mm, 34 parts, among them J1 PJ-644F, J10 Conn_01x03, J11 Conn_01x03, J12 Conn_01x03, J13 Conn_01x03, J14 Conn_01x03, J15 Conn_01x03, J16 Conn_01x04, J17 PJ-202A, J2 Conn_01x06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

Commit message: Add files via upload
Parts:
- added D3: TVS, Diode_THT:D_DO-15_P12.70mm_Horizontal, F.Cu at (80.5, 51.2)
Routing:
- net VCC: track 171.8 -> 165.8 mm
