File: KiCad/Guitar_Fx_Dev.kicad_sch (KiCad schematic)
At the start: 33 parts, among them J1 PJ-644F, J10 Conn_01x03, J11 Conn_01x03, J12 Conn_01x03, J13 Conn_01x03, J14 Conn_01x03, J15 Conn_01x03, J16 Conn_01x04, J17 PJ-202A, J2 Conn_01x06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

Commit message: Add files via upload
Parts:
- added D3: TVS, Diode_THT:D_DO-15_P12.70mm_Horizontal, symbol Diode:1.5KExxA
Connections:
- net GNDREF: now also D3.2 (A2)
- net VCC: now also D3.1 (A1)
Other:
- note added: "Optional V Spike Protection"
- moved on the sheet: C3
Changed lines of the file:
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@@
 	)
 	(junction
-		(at 46.99 168.91)
+		(at 39.37 168.91)
 		(diameter 0)
 		(color 0 0 0 0)
@@
 	)
 	(junction
+		(at 54.61 168.91)
+		(diameter 0)
+		(color 0 0 0 0)
+	)
+	(junction
 		(at 105.41 168.91)
 		(diameter 0)
@@
 	(wire
 		(pts
-			(xy 46.99 173.99) (xy 46.99 168.91)
+			(xy 54.61 173.99) (xy 54.61 168.91)
 		)
 		(stroke
@@
 	(wire
 		(pts
-			(xy 46.99 181.61) (xy 46.99 179.07)
+			(xy 54.61 181.61) (xy 54.61 179.07)
 		)
 		(stroke
@@
 	(wire
 		(pts
+			(xy 39.37 168.91) (xy 54.61 168.91)
+		)
+		(stroke
+			(width 0)
+			(type default)
+		)
+	)
+	(wire
+		(pts
 			(xy 180.34 129.54) (xy 165.1 129.54)
 		)
@@
 	(wire
 		(pts
-			(xy 46.99 168.91) (xy 46.99 160.02)
+			(xy 39.37 168.91) (xy 39.37 160.02)
 		)
 		(stroke
@@
 	(wire
 		(pts
-			(xy 46.99 168.91) (xy 62.23 168.91)
-		)
-		(stroke
-			(width 0)
-			(type default)
-		)
-	)
-	(wire
-		(pts
 			(xy 109.22 35.56) (xy 113.03 35.56)
 		)
@@
 	(wire
 		(pts
+			(xy 39.37 180.34) (xy 39.37 181.61)
+		)
+		(stroke
+			(width 0)
+			(type default)
+		)
+	)
+	(wire
+		(pts
 			(xy 109.22 25.4) (xy 116.84 25.4)
 		)
@@
 	(wire
 		(pts
+			(xy 39.37 168.91) (xy 39.37 172.72)
+		)
+		(stroke
+			(width 0)
+			(type default)
+		)
+	)
+	(wire
+		(pts
 			(xy 236.22 102.87) (xy 236.22 105.41)
 		)
@@
 	(wire
 		(pts
+			(xy 54.61 168.91) (xy 62.23 168.91)
+		)
+		(stroke
+			(width 0)
+			(type default)
+		)
+	)
+	(wire
+		(pts
 			(xy 88.9 173.99) (xy 88.9 176.53)
 		)
@@
 	(wire
 		(pts
-			(xy 33.02 168.91) (xy 46.99 168.91)
+			(xy 33.02 168.91) (xy 39.37 168.91)
 		)
 		(stroke
@@
 	(text "+9v"
 		(exclude_from_sim no)
-		(at 45.72 156.21 0)
+		(at 37.084 156.718 0)
 		(effects
 			(font
@@
 		)
 	)
+	(text "Optional \nV Spike\nProtection"
+		(exclude_from_sim no)
+		(at 41.402 184.912 0)
+		(effects
+			(font
+				(size 1.27 1.27)
+			)
+			(justify left bottom)
+		)
+	)
 	(text "Tip_n"
 		(exclude_from_sim no)
@@
 	(symbol
 		(lib_id "Guitar_Fx_Dev-rescue:CP1_Small-Device")
-		(at 46.99 176.53 0)
+		(at 54.61 176.53 0)
 		(unit 1)
 		(exclude_from_sim no)
@@
 		(dnp no)
 		(property "Reference" "C3"
-			(at 50.673 176.276 0)
+			(at 58.293 176.276 0)
 			(effects
 				(font
@@
 		)
 		(property "Value" "10uF"
-			(at 51.435 178.435 0)
+			(at 59.055 178.435 0)
 			(effects
 				(font
@@
 		)
 		(property "Footprint" "Capacitor_THT:CP_Radial_D5.0mm_P2.50mm"
-			(at 46.99 176.53 0)
+			(at 54.61 176.53 0)
 			(effects
 				(font
@@
 		)
 		(property "Datasheet" "~"
-			(at 46.99 176.53 0)
+			(at 54.61 176.53 0)
 			(effects
 				(font
@@
 		)
 		(property "Description" ""
-			(at 46.99 176.53 0)
+			(at 54.61 176.53 0)
 			(effects
 				(font
@@
 	(symbol
 		(lib_id "Guitar_Fx_Dev-rescue:VCC-power")
-		(at 46.99 160.02 0)
+		(at 39.37 160.02 0)
 		(unit 1)
 		(exclude_from_sim no)
@@
 		(dnp no)
 		(property "Reference" "#PWR06"
-			(at 46.99 163.83 0)
+			(at 39.37 163.83 0)
 			(effects
 				(font
@@
 		)
 		(property "Value" "VCC"
-			(at 47.4218 155.6258 0)
+			(at 39.8018 155.6258 0)
 			(effects
 				(font
@@
 		)
 		(property "Footprint" ""
-			(at 46.99 160.02 0)
+			(at 39.37 160.02 0)
 			(effects
 				(font
@@
 		)
 		(property "Datasheet" ""
-			(at 46.99 160.02 0)
+			(at 39.37 160.02 0)
 			(effects
 				(font
@@
 		)
 		(property "Description" ""
-			(at 46.99 160.02 0)
+			(at 39.37 160.02 0)
 			(effects
 				(font
@@
 	(symbol
 		(lib_id "Guitar_Fx_Dev-rescue:GNDREF-power")
-		(at 46.99 181.61 0)
+		(at 54.61 181.61 0)
 		(unit 1)
 		(exclude_from_sim no)
@@
 		(dnp no)
 		(property "Reference" "#PWR017"
-			(at 46.99 187.96 0)
+			(at 54.61 187.96 0)
 			(effects
 				(font
@@
 		)
 		(property "Value" "GNDREF"
-			(at 47.117 186.0042 0)
+			(at 54.737 186.0042 0)
 			(effects
 				(font
@@
 		)
 		(property "Footprint" ""
-			(at 46.99 181.61 0)
+			(at 54.61 181.61 0)
 			(effects
 				(font
@@
 		)
 		(property "Datasheet" ""
-			(at 46.99 181.61 0)
+			(at 54.61 181.61 0)
 			(effects
 				(font
@@
 		)
 		(property "Description" ""
-			(at 46.99 181.61 0)
+			(at 54.61 181.61 0)
 			(effects
 				(font
@@
 	)
 	(symbol
+		(lib_id "Guitar_Fx_Dev-rescue:GNDREF-power")
+		(at 39.37 181.61 0)
+		(unit 1)
+		(exclude_from_sim no)
+		(in_bom yes)
+		(on_board yes)
+		(dnp no)
+		(property "Reference" "#PWR019"
+			(at 39.37 187.96 0)
+			(effects
+				(font
+					(size 1.27 1.27)
+				)
+				(hide yes)
+			)
+		)
+		(property "Value" "GNDREF"
+			(at 39.497 186.0042 0)
+			(effects
+				(font
+					(size 1.27 1.27)
+				)
+				(hide yes)
+			)
+		)
+		(property "Footprint" ""
+			(at 39.37 181.61 0)
+			(effects
+				(font
+					(size 1.27 1.27)
+				)
+				(hide yes)
+			)
+		)
+		(property "Datasheet" ""
+			(at 39.37 181.61 0)
+			(effects
+				(font
+					(size 1.27 1.27)
+				)
+				(hide yes)
+			)
+		)
+		(property "Description" ""
+			(at 39.37 181.61 0)
+			(effects
+				(font
+					(size 1.27 1.27)
+				)
+				(hide yes)
+			)
+		)
+		(pin "1"
+		)
+		(instances
+			(project "Guitar_Fx_Dev"
+				(path "/1b077fc9-b8d8-443a-8fee-1b5107551db8"
+					(reference "#PWR019")
+					(unit 1)
+				)
+			)
+		)
+	)
+	(symbol
 		(lib_id "Device:C_Small")
 		(at 96.52 171.45 180)
@@
 					(unit 1)
 				)
+			)
+		)
+	)
+	(symbol
+		(lib_id "Diode:1.5KExxA")
+		(at 39.37 176.53 270)
+		(unit 1)
+		(exclude_from_sim no)
+		(in_bom yes)
+		(on_board yes)
+		(dnp no)
+		(property "Reference" "D3"
+			(at 41.91 175.2599 90)
+			(effects
+				(font
+					(size 1.27 1.27)
+				)
+				(justify left)
+			)
+		)
+		(property "Value" "TVS"
+			(at 41.656 177.2919 90)
+			(effects
+				(font
+					(size 1.27 1.27)
+				)
+				(justify left)
+			)
+		)
+		(property "Footprint" "Diode_THT:D_DO-15_P12.70mm_Horizontal"
+			(at 34.29 176.53 0)
+			(effects
+				(font
+					(size 1.27 1.27)
+				)
+				(hide yes)
+			)
+		)
+		(property "Datasheet" "https://www.vishay.com/docs/88301/15ke.pdf"
+			(at 39.37 175.26 0)
+			(effects
+				(font
+					(size 1.27 1.27)
+				)
+				(hide yes)
+			)
+		)
+		(property "Description" "1500W unidirectional TVS diode, DO-201AE"
+			(at 39.37 176.53 0)
+			(effects
+				(font
+					(size 1.27 1.27)
+				)
+				(hide yes)
+			)
+		)
+		(pin "1"
+		)
+		(pin "2"
+		)
+		(instances
+			(project ""
+				(path "/1b077fc9-b8d8-443a-8fee-1b5107551db8"
+					(reference "D3")
+					(unit 1)
+				)
